File: PCB/gps_tracer.kicad_sch (KiCad schematic)
At the start: 86 parts, among them IC1 TC4056A, J1 Mic, J2 SPK, J3 sensor, J4 BATTERY, J5 Micro_SD_Card, P1 USB_C_Plug_USB2.0, Q1 S8050, Q2 S8050, Q3 FDN358P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

Commit message: The PCB was traced, and ordered
Parts:
- removed H1, H2, H3, H4: MountingHole, MountingHole:MountingHole_2.2mm_M2, symbol Mechanical:MountingHole
- added C6 (x3): 100n, Capacitor_SMD:C_0603_1608Metric_Pad1.08x0.95mm_HandSolder, symbol Device:C
- added C6: 22u, Capacitor_SMD:C_0805_2012Metric_Pad1.18x1.45mm_HandSolder, symbol Device:C
- added R15 (x2): ????, Resistor_SMD:R_0603_1608Metric_Pad0.98x0.95mm_HandSolder, symbol Device:R
- C6: footprint Capacitor_SMD:C_0603_1608Metric_Pad1.08x0.95mm_HandSolder -> Capacitor_SMD:C_0805_2012Metric_Pad1.18x1.45mm_HandSolder
- D2, D8, D9: footprint LED_SMD:LED_0805_2012Metric_Pad1.15x1.40mm_HandSolder -> LED_SMD:LED_0603_1608Metric_Pad1.05x0.95mm_HandSolder
- J1, J2, J4: footprint Connector_PinHeader_1.27mm:PinHeader_1x02_P1.27mm_Vertical -> Footprint_library:JST 1.25
- J3: value sensor -> I2C; footprint Connector_JST:JST_EH_B4B-EH-A_1x04_P2.50mm_Vertical -> Connector_PinHeader_1.27mm:PinHeader_1x04_P1.27mm_Vertical
- L1: footprint (none) -> Inductor_SMD:L_Ferrocore_DLG-0703
Connections:
- net +3.3V: now also U12.13 (VDD), U12.8 (VLOGIC), C6.2
- net GND: now also U12.1 (CLKIN), U12.11 (FSYNC), U12.18 (GND), U12.9 (AD0), U7.5 (GND), C6.1, C6.1, C6.1; no longer U7.6 (GND)
- net MPU5060_INT: now also U4.6 (IO34)
- net RST_GSM: now also U4.8 (IO32), U7.2 (RST); no longer U7.3 (RST)
- net RXD_GSM: now also U7.3 (RXD); no longer U7.4 (RXD)
- net TXD_GSM: now also U7.4 (TXD); no longer U7.5 (TXD)
- net at U12.10 (REGOUT): now also C6.2
- net at U12.20 (CPOUT): now also C6.2
- net at J2.1 (Pin_1): now also U7.6 (SPKM); no longer U7.7 (SPKM)
- net at J2.2 (Pin_2): now also U7.7 (SPKN); no longer U7.8 (SPKN)
- net BATTERY_VOLTAGE: now reaches U4.7 (IO35)
- net BATTERY_VOLTAGE: now also R15.1, R15.2
- net at C6.2, J4.1 (Pin_1), U8.2 (S1)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: now also C6.2, R15.2
- net at C6.1, IC1.5 (BAT), Q4.3 (D)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: now also J4.2 (Pin_2), R15.1, C6.1, R15.1; no longer C6.1, R15.2, U9.5 (VCC)
- net at U7.1 (VCC): now also C5.1, C5.1, Q8.3 (D)
- net at U7.10 (DTR): no longer J1.2 (Pin_2)
- net at J1.1 (Pin_1): now also U7.8 (MICN); no longer U7.9 (MICN)
- new net: C6.1, R15.2, U9.5 (VCC)
- new net: J1.2 (Pin_2), U7.9 (MICP)
- no-connect marks 38 -> 37
Other:
- note added: "Додатифутпрінт на дросель"
- note added: "Які значення резисторів дільників напруги?"
- note removed: "!!!!!!!!!!!!!"
- note removed: "ВИМІРЮВАТИ НАПРУНУ !!!!!!!!!!!!!!!!!!!!!!"
- note removed: "Додати аналогову схему вимярювання напруги на батереї"
- note removed: "ЗАБРАТИ НОЖКУ NET!!!"
- moved on the sheet: AE1, C5, J1, J2, J4, Q3, Q8, R15, U6
